File: electronics/teensy-board.sch (EAGLE design)
At the start: 21 parts

Commit message: fixed flipped charlieplexed led
Changed lines of the file:
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@@
 <instance part="R8" gate="G$1" x="15.24" y="5.08"/>
 <instance part="R9" gate="G$1" x="45.72" y="5.08"/>
-<instance part="U$7" gate="G$1" x="2.54" y="-30.48"/>
+<instance part="U$7" gate="G$1" x="20.32" y="86.36"/>
 </instances>
 <busses>
